File: springreverb_lm386.kicad_sch (KiCad schematic)
At the start: 61 parts, among them J1 IN, J10 To2, J11 To_Tank, J12 From_Tank, J13 FromGND, J14 From, J15 VR2_3, J16 VR2_3GND, J17 OUT, J2 INGND, J3 GND, J4 Vin, J5 VR1_3, J6 VR1_2, J7 VR3_1, J8 ToGND, J9 To, U1 TL072, U2 TC1044S, U3 4556ADD

Commit message: 一旦回路完成
Parts:
- removed C16, C19: 100u, Capacitor_THT:CP_Radial_D6.3mm_P2.50mm, symbol Device:C_Small_US
- removed C17, C18: 0.1u, Capacitor_THT:C_Rect_L4.0mm_W2.5mm_P2.50mm, symbol Device:C_Small
- removed J6: VR1_2, MyLibrary:PinHeader_1x01_P2.54mm_Vertical, symbol Connector:Conn_01x01_Pin
- removed R12: 47, Resistor_THT:R_Axial_DIN0204_L3.6mm_D1.6mm_P7.62mm_Horizontal, symbol Device:R_Small
- removed R16: 1k, Resistor_THT:R_Axial_DIN0204_L3.6mm_D1.6mm_P2.54mm_Vertical, symbol Device:R_Small
- removed R5: 1.2k, Resistor_THT:R_Axial_DIN0204_L3.6mm_D1.6mm_P2.54mm_Vertical, symbol Device:R_Small
- removed R7: 10, Resistor_THT:R_Axial_DIN0204_L3.6mm_D1.6mm_P7.62mm_Horizontal, symbol Device:R_Small
- removed R9: 100, Resistor_THT:R_Axial_DIN0204_L3.6mm_D1.6mm_P7.62mm_Horizontal, symbol Device:R_Small
- removed U3: 4556ADD, MyLibrary:CERDIP-8_W7.62mm_SideBrazed_Socket, symbol Amplifier_Operational:TL072
- added C11: 100u, Capacitor_THT:CP_Radial_D10.0mm_P2.50mm, symbol Device:C_Small_US
- added C14: 0.047u, Capacitor_THT:C_Rect_L10.3mm_W5.0mm_P7.50mm_MKS4, symbol Device:C_Small
- added C15: 100u, Capacitor_THT:CP_Radial_D7.5mm_P2.50mm, symbol Device:C_Small_US
- added C7: 0.22u, MyLibrary:10.5_5.0_p7.5, symbol Device:C_Small
- added C9: 10u, Capacitor_THT:CP_Radial_D6.3mm_P2.50mm, symbol Device:C_Small_US
- added J11: VR_2_2, MyLibrary:PinHeader_1x01_P2.54mm_Vertical, symbol Connector:Conn_01x01_Pin
- added J12: VR_2GND, MyLibrary:PinHeader_1x01_P2.54mm_Vertical, symbol Connector:Conn_01x01_Pin
- added J14: FromSW, MyLibrary:PinHeader_1x01_P2.54mm_Vertical, symbol Connector:Conn_01x01_Pin
- added J5: LEDGND, MyLibrary:PinHeader_1x01_P2.54mm_Vertical, symbol Connector:Conn_01x01_Pin
- added J7: toC6, MyLibrary:PinHeader_1x01_P2.54mm_Vertical, symbol Connector:Conn_01x01_Pin
- added J9: FromC, MyLibrary:PinHeader_1x01_P2.54mm_Vertical, symbol Connector:Conn_01x01_Pin
- added R6: 10, Resistor_THT:R_Axial_DIN0204_L3.6mm_D1.6mm_P7.62mm_Horizontal, symbol Device:R_Small
- added SW1: SW_SPDT, symbol Switch:SW_SPDT
- added SW2: SW_SPST, symbol Switch:SW_SPST
- added U3: LM386, MyLibrary:CERDIP-8_W7.62mm_SideBrazed_Socket, symbol Amplifier_Audio:LM386
- added VR2: B1k, symbol Device:R_Potentiometer
- C12: renamed from C9; footprint Capacitor_THT:CP_Radial_D10.0mm_P5.00mm -> Capacitor_THT:CP_Radial_D13.0mm_P5.00mm
- C16: renamed from C11; footprint Capacitor_THT:CP_Radial_D6.3mm_P2.50mm -> Capacitor_THT:CP_Radial_D7.5mm_P2.50mm
- C19: renamed from C14; footprint Capacitor_THT:CP_Radial_D6.3mm_P2.50mm -> Capacitor_THT:CP_Radial_D7.5mm_P2.50mm
- C2: footprint MyLibrary:10.5_5.0_p7.5 -> Capacitor_THT:C_Rect_L10.3mm_W5.0mm_P7.50mm_MKS4
- C3: footprint Capacitor_THT:CP_Radial_D10.0mm_P5.00mm -> Capacitor_THT:CP_Radial_D13.0mm_P5.00mm
- C4: renamed from C5; footprint Capacitor_THT:CP_Radial_D6.3mm_P2.50mm -> Capacitor_THT:CP_Radial_D7.5mm_P2.50mm
- C6: value 560p -> 0.1u; footprint (none) -> MyLibrary:10.5_5.0_p7.5
- J10: value To2 -> VR2_3
- J8: value ToGND -> toC7
- renumbered C8 to C10, C10 to C13, C12 to C17, C13 to C18, C15 to C20, C20 to C21, C4 to C5, C7 to C8, J9 to J13, J11 to J15, J12 to J16, J13 to J17, J14 to J18, J15 to J19, J16 to J20, J7 to J21, J17 to J22, J5 to J6, R15 to R10, R8 to R4, R10 to R5, R11 to R7, R13 to R8, R14 to R9, VR2 to VR3, VR3 to VR4
Connections:
- net GND: now also C11.2, J12.1 (Pin_1), J14.1 (Pin_1), J5.1 (Pin_1), J9.1 (Pin_1), R6.2, SW2.1 (A), U3.2 (-), U3.4 (GND); no longer J8.1 (Pin_1)
- net at VR1.2: now also SW1.2 (B)
- net at J13.1 (Pin_1), J15.1 (In): now also C15.2; no longer C6.2
- net at J4.1 (Pin_1), R3.2, U2.1 (BOOST)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: now also U3.6 (V+)
- new net: C9.1, U3.1 (GAIN)
- new net: C9.2, J10.1 (Pin_1), VR2.3
- new net: C6.2, J7.1 (Pin_1), SW1.1 (A)
- new net: J11.1 (Pin_1), U3.8 (GAIN), VR2.1, VR2.2
- new net: C6.1, C7.1, U3.3 (+)
- new net: C14.2, C15.1, U3.5
- new net: C11.1, U3.7 (BYPASS)
- new net: C7.2, J8.1 (Pin_1), SW1.3 (C)
- new net: J15.2 (Ext), SW2.2 (B)
- new net: C14.1, R6.1
Other:
- moved on the sheet: C20, C21, J13, J15, J16, J17, J18, J19, J20, J21, J22, R10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
